File: w4/s-ispv2.brd (EAGLE design)
At the start: 46.4 x 18 mm, 22 parts, among them IC1 ATTINY44-SSU, J1 SJ, J2 SJ, X1 USBPCB, X2 AVRISPSMD

Commit message: s-isp-v2
Parts:
- removed C1, C2: 8p, rcl:C1206
- removed C3: 0.1u, rcl:C1206
- removed J1, J2: SJ, fab:SJFAB
- removed R5: 0, rcl:R1206
- removed XTAL1: 20MHz, fab:2-SMD-5X3MM
- added U$1: RESONATOR, fab:EFOBM
- moved R8 22.8 mm to (22.6, 1.54), turned to 0 degrees
- moved LED2 18.4 mm to (28.4, 4.11), turned to 180 degrees
- moved LED1 17.2 mm to (28.4, 1.51), turned to 180 degrees
- moved R7 11.2 mm to (35.7, 3.77), turned to 0 degrees
- moved C4 2.01 mm to (18.6, 3.53)
- moved X2 1.03 mm to (36.1, 11.4), turned to 270 degrees
- moved IC1 1.00 mm to (24.9, 12.3)
Connections:
- removed net N$3: J1.2, R5.2
- removed net N$4: J2.1, X2.2
- removed net N$5: IC1.4, R4.1, R5.1
- net GND: now also U$1.2; no longer C1.2, C2.2, C3.2
- net RST: now also IC1.4, R4.1; no longer J1.1
- net VCC: now also X2.2; no longer C3.1, J2.2
- net XTAL1: now also U$1.3; no longer C1.1, XTAL1.P$2
- net XTAL2: now also U$1.1; no longer C2.1, XTAL1.P$1
Routing:
- net GND: track 102.0 -> 62.0 mm
- net RST: track 11.6 -> 33.1 mm, vias 0 -> 2
- net N$5: track 20.6 -> 0.00 mm
- net MISO: track 8.60 -> 24.2 mm
- net N$4: track 15.0 -> 0.00 mm
- net XTAL2: track 18.0 -> 4.57 mm
- net VCC: track 47.8 -> 57.3 mm
- net N$3: track 6.07 -> 0.00 mm
- net XTAL1: track 8.34 -> 4.22 mm
- net SCK: track 8.84 -> 11.7 mm
- net MOSI: track 21.1 -> 23.2 mm
- net N$7: track 2.07 -> 3.02 mm
- net D-: track 11.8 -> 11.2 mm
- net N$1: track 15.9 -> 15.4 mm
Other:
- board size 46.4 x 18 mm -> 40 x 17.9 mm
