File: w4/s-ispv2.sch (EAGLE design)
At the start: 22 parts, among them IC1 ATTINY44-SSU, J1 SJ, J2 SJ, X1 USBPCB, X2 AVRISPSMD

Commit message: s-isp-v2
Parts:
- removed C1, C2: 8p, rcl:C-USC1206
- removed C3: 0.1u, rcl:C-USC1206
- removed J1, J2: SJ, fab:SOLDER_JUMPER
- removed R5: 0, rcl:R-US_R1206
- removed XTAL1: 20MHz, fab:CRYSTAL
- added U$1: RESONATOR, fab:RESONATOR
Connections:
- removed net N$3: J1.2, R5.2
- removed net N$4: J2.1, X2.VCC
- removed net N$5: IC1.(PCINT11/RESET/DW)PB3, R4.1, R5.1
- net GND: now also U$1.2; no longer C1.2, C2.2, C3.2
- net RST: now also IC1.(PCINT11/RESET/DW)PB3, R4.1; no longer J1.1
- net VCC: now also X2.VCC; no longer C3.1, J2.2
- net XTAL1: now also U$1.3; no longer C1.1, XTAL1.2
- net XTAL2: now also U$1.1; no longer C2.1, XTAL1.1
Other:
- moved on the sheet: C4
Changed lines of the file:
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@@
 <part name="R4" library="rcl" deviceset="R-US_" device="R1206" value="10K"/>
 <part name="SUPPLY8" library="supply2" deviceset="VCC" device=""/>
-<part name="J2" library="fab" deviceset="SOLDER_JUMPER" device="" value="SJ"/>
-<part name="C1" library="rcl" deviceset="C-US" device="C1206" value="8p"/>
-<part name="C2" library="rcl" deviceset="C-US" device="C1206" value="8p"/>
 <part name="SUPPLY9" library="supply2" deviceset="GND" device=""/>
-<part name="C3" library="rcl" deviceset="C-US" device="C1206" value="0.1u"/>
 <part name="C4" library="rcl" deviceset="C-US" device="C1206" value="1u"/>
 <part name="SUPPLY10" library="supply2" deviceset="VCC" device=""/>
 <part name="SUPPLY11" library="supply2" deviceset="GND" device=""/>
-<part name="XTAL1" library="fab" deviceset="CRYSTAL" device="" value="20MHz"/>
 <part name="FRAME1" library="frames" deviceset="LETTER_L" device=""/>
 <part name="R6" library="rcl" deviceset="R-US_" device="R1206" value="499"/>
-<part name="R5" library="rcl" deviceset="R-US_" device="R1206" value="0"/>
-<part name="J1" library="fab" deviceset="SOLDER_JUMPER" device="" value="SJ"/>
 <part name="R7" library="rcl" deviceset="R-US_" device="R1206" value="499"/>
 <part name="R8" library="rcl" deviceset="R-US_" device="R1206" value="499"/>
@@
 <part name="LED2" library="led" deviceset="LED" device="SMT1206"/>
 <part name="SUPPLY12" library="supply2" deviceset="GND" device=""/>
+<part name="U$1" library="fab" deviceset="RESONATOR" device=""/>
 </parts>
 <sheets>
@@
 <instance part="R4" gate="G$1" x="111.76" y="106.68" rot="R90"/>
 <instance part="SUPPLY8" gate="G$1" x="111.76" y="116.84"/>
-<instance part="J2" gate="G$1" x="160.02" y="127"/>
-<instance part="C1" gate="G$1" x="205.74" y="91.44" rot="R90"/>
-<instance part="C2" gate="G$1" x="205.74" y="81.28" rot="R90"/>
-<instance part="SUPPLY9" gate="GND" x="213.36" y="73.66"/>
-<instance part="C3" gate="G$1" x="187.96" y="124.46"/>
-<instance part="C4" gate="G$1" x="195.58" y="124.46"/>
+<instance part="SUPPLY9" gate="GND" x="220.98" y="73.66"/>
+<instance part="C4" gate="G$1" x="187.96" y="124.46"/>
 <instance part="SUPPLY10" gate="G$1" x="187.96" y="134.62"/>
 <instance part="SUPPLY11" gate="GND" x="187.96" y="111.76"/>
-<instance part="XTAL1" gate="G$1" x="200.66" y="86.36" rot="R90"/>
 <instance part="FRAME1" gate="G$1" x="0" y="0"/>
 <instance part="FRAME1" gate="G$2" x="147.32" y="0"/>
 <instance part="R6" gate="G$1" x="40.64" y="121.92" rot="R90"/>
-<instance part="R5" gate="G$1" x="106.68" y="99.06" rot="R180"/>
-<instance part="J1" gate="G$1" x="93.98" y="99.06"/>
 <instance part="R7" gate="G$1" x="81.28" y="86.36" rot="R90"/>
 <instance part="R8" gate="G$1" x="71.12" y="76.2" rot="R90"/>
@@
 <instance part="LED2" gate="G$1" x="81.28" y="76.2"/>
 <instance part="SUPPLY12" gate="GND" x="71.12" y="68.58"/>
+<instance part="U$1" gate="G$1" x="210.82" y="86.36" rot="R90"/>
 </instances>
 <busses>
@@
 </segment>
 <segment>
-<wire x1="165.1" y1="127" x2="167.64" y2="127" width="0.1524" layer="91"/>
 <wire x1="167.64" y1="127" x2="167.64" y2="132.08" width="0.1524" layer="91"/>
-<pinref part="J2" gate="G$1" pin="2"/>
 <pinref part="SUPPLY2" gate="G$1" pin="VCC"/>
-</segment>
-<segment>
-<wire x1="187.96" y1="132.08" x2="187.96" y2="129.54" width="0.1524" layer="91"/>
-<wire x1="187.96" y1="129.54" x2="187.96" y2="127" width="0.1524" layer="91"/>
-<wire x1="195.58" y1="127" x2="195.58" y2="129.54" width="0.1524" layer="91"/>
-<wire x1="195.58" y1="129.54" x2="187.96" y2="129.54" width="0.1524" layer="91"/>
-<junction x="187.96" y="129.54"/>
+<pinref part="X2" gate="G$1" pin="VCC"/>
+<wire x1="144.78" y1="127" x2="167.64" y2="127" width="0.1524" layer="91"/>
+</segment>
+<segment>
+<wire x1="187.96" y1="132.08" x2="187.96" y2="127" width="0.1524" layer="91"/>
 <pinref part="SUPPLY10" gate="G$1" pin="VCC"/>
-<pinref part="C3" gate="G$1" pin="1"/>
 <pinref part="C4" gate="G$1" pin="1"/>
 </segment>
@@
 </segment>
 <segment>
-<wire x1="210.82" y1="91.44" x2="213.36" y2="91.44" width="0.1524" layer="91"/>
-<wire x1="213.36" y1="91.44" x2="213.36" y2="81.28" width="0.1524" layer="91"/>
-<wire x1="213.36" y1="81.28" x2="213.36" y2="76.2" width="0.1524" layer="91"/>
-<wire x1="210.82" y1="81.28" x2="213.36" y2="81.28" width="0.1524" layer="91"/>
-<junction x="213.36" y="81.28"/>
-<pinref part="C1" gate="G$1" pin="2"/>
 <pinref part="SUPPLY9" gate="GND" pin="GND"/>
-<pinref part="C2" gate="G$1" pin="2"/>
-</segment>
-<segment>
-<wire x1="187.96" y1="114.3" x2="187.96" y2="116.84" width="0.1524" layer="91"/>
-<wire x1="187.96" y1="116.84" x2="187.96" y2="119.38" width="0.1524" layer="91"/>
-<wire x1="195.58" y1="119.38" x2="195.58" y2="116.84" width="0.1524" layer="91"/>
-<wire x1="195.58" y1="116.84" x2="187.96" y2="116.84" width="0.1524" layer="91"/>
-<junction x="187.96" y="116.84"/>
+<pinref part="U$1" gate="G$1" pin="2"/>
+<wire x1="218.44" y1="86.36" x2="220.98" y2="86.36" width="0.1524" layer="91"/>
+<wire x1="220.98" y1="86.36" x2="220.98" y2="76.2" width="0.1524" layer="91"/>
+</segment>
+<segment>
+<wire x1="187.96" y1="114.3" x2="187.96" y2="119.38" width="0.1524" layer="91"/>
 <pinref part="SUPPLY11" gate="GND" pin="GND"/>
-<pinref part="C3" gate="G$1" pin="2"/>
 <pinref part="C4" gate="G$1" pin="2"/>
 </segment>
@@
 <wire x1="88.9" y1="99.06" x2="81.28" y2="99.06" width="0.1524" layer="91"/>
 <label x="81.28" y="99.06" size="1.778" layer="95"/>
-<pinref part="J1" gate="G$1" pin="1"/>
+</segment>
+<segment>
+<wire x1="114.3" y1="99.06" x2="111.76" y2="99.06" width="0.1524" layer="91"/>
+<wire x1="111.76" y1="99.06" x2="111.76" y2="101.6" width="0.1524" layer="91"/>
+<pinref part="IC1" gate="1" pin="(PCINT11/RESET/DW)PB3"/>
+<pinref part="R4" gate="G$1" pin="1"/>
+<wire x1="99.06" y1="99.06" x2="111.76" y2="99.06" width="0.1524" layer="91"/>
+<junction x="111.76" y="99.06"/>
 </segment>
 </net>
@@
 </segment>
 </net>
-<net name="N$4" class="0">
-<segment>
-<wire x1="144.78" y1="127" x2="154.94" y2="127" width="0.1524" layer="91"/>
-<pinref part="X2" gate="G$1" pin="VCC"/>
-<pinref part="J2" gate="G$1" pin="1"/>
-</segment>
-</net>
 <net name="XTAL1" class="0">
 <segment>
-<wire x1="203.2" y1="91.44" x2="200.66" y2="91.44" width="0.1524" layer="91"/>
-<wire x1="200.66" y1="91.44" x2="190.5" y2="91.44" width="0.1524" layer="91"/>
-<wire x1="200.66" y1="88.9" x2="200.66" y2="91.44" width="0.1524" layer="91"/>
-<junction x="200.66" y="91.44"/>
 <label x="190.5" y="91.44" size="1.778" layer="95"/>
-<pinref part="C1" gate="G$1" pin="1"/>
-<pinref part="XTAL1" gate="G$1" pin="2"/>
+<pinref part="U$1" gate="G$1" pin="3"/>
+<wire x1="190.5" y1="93.98" x2="210.82" y2="93.98" width="0.1524" layer="91"/>
 </segment>
 <segment>
@@
 <net name="XTAL2" class="0">
 <segment>
-<wire x1="203.2" y1="81.28" x2="200.66" y2="81.28" width="0.1524" layer="91"/>
-<wire x1="200.66" y1="81.28" x2="190.5" y2="81.28" width="0.1524" layer="91"/>
-<wire x1="200.66" y1="83.82" x2="200.66" y2="81.28" width="0.1524" layer="91"/>
-<junction x="200.66" y="81.28"/>
-<label x="190.5" y="81.28" size="1.778" layer="95"/>
-<pinref part="C2" gate="G$1" pin="1"/>
-<pinref part="XTAL1" gate="G$1" pin="1"/>
+<label x="190.5" y="78.74" size="1.778" layer="95"/>
+<wire x1="190.5" y1="78.74" x2="210.82" y2="78.74" width="0.1524" layer="91"/>
+<pinref part="U$1" gate="G$1" pin="1"/>
 </segment>
 <segment>
@@
 </segment>
 </net>
-<net name="N$5" class="0">
-<segment>
-<wire x1="114.3" y1="99.06" x2="111.76" y2="99.06" width="0.1524" layer="91"/>
-<wire x1="111.76" y1="99.06" x2="111.76" y2="101.6" width="0.1524" layer="91"/>
-<junction x="111.76" y="99.06"/>
-<pinref part="IC1" gate="1" pin="(PCINT11/RESET/DW)PB3"/>
-<pinref part="R4" gate="G$1" pin="1"/>
-<pinref part="R5" gate="G$1" pin="1"/>
-</segment>
-</net>
 <net name="N$6" class="0">
 <segment>
@@
 </segment>
 </net>
-<net name="N$3" class="0">
-<segment>
-<wire x1="99.06" y1="99.06" x2="101.6" y2="99.06" width="0.1524" layer="91"/>
-<pinref part="R5" gate="G$1" pin="2"/>
-<pinref part="J1" gate="G$1" pin="2"/>
-</segment>
-</net>
