File: w10/gest-mod.brd (EAGLE design)
At the start: 49 x 55.7 mm, 25 parts, among them IC2 ATMEGA88-THIN, IC6 75176AD, IC8 TL780_VREG, J2 AVR-7_AVR-ISP-6VERT, J3 KK-4P, J9 22-27-2021-02

Commit message: sibu:- update gest
Routing:
- net RS485-A: track 37.0 -> 37.8 mm
Other:
- board size 49 x 55.7 mm -> 49.8 x 56.5 mm
