File: w11/ss-test-rev1.brd (EAGLE design)
At the start: 38 x 56.6 mm, 17 parts, among them J1 CON-MOLEX_22-27-2041-04

Commit message: w11 reset pullup
Parts:
- added R3: 10k, fab:R1206FAB
Connections:
- net RST: now also R3.1
- net VCC: now also R3.2
Routing:
- net RST: track 8.93 -> 12.8 mm
- net N$19: track 13.0 -> 9.71 mm, vias 2 -> 1
- net VCC: track 145.6 -> 147.4 mm
Changed lines of the file:
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@@
 <element name="R1" library="fab" package="R1206FAB" value="499" x="55.88" y="39.37" rot="R270"/>
 <element name="R2" library="fab" package="R1206FAB" value="499" x="35.6" y="36.7"/>
+<element name="R3" library="fab" package="R1206FAB" value="10k" x="43" y="52.5" rot="R90"/>
 </elements>
 <signals>
@@
 <wire x1="40.73" y1="46.9" x2="40.64" y2="46.99" width="0.6096" layer="1"/>
 <wire x1="44.45" y1="46.95" x2="44.41" y2="46.99" width="0.8128" layer="1"/>
-<wire x1="44.41" y1="46.99" x2="40.64" y2="46.99" width="0.8128" layer="1"/>
+<wire x1="44.41" y1="46.99" x2="43.1" y2="46.99" width="0.8128" layer="1"/>
+<contactref element="R3" pad="1"/>
+<wire x1="43.1" y1="46.99" x2="40.64" y2="46.99" width="0.8128" layer="1"/>
+<wire x1="43" y1="50.849" x2="43.1" y2="50.749" width="0.8128" layer="1"/>
+<wire x1="43.1" y1="50.749" x2="43.1" y2="46.99" width="0.8128" layer="1"/>
 </signal>
 <signal name="SCK">
@@
 <wire x1="58.7" y1="48" x2="58.7" y2="51" width="0.6096" layer="1"/>
 <wire x1="58.7" y1="51" x2="53.8" y2="55.9" width="0.6096" layer="1"/>
-<wire x1="53.8" y1="55.9" x2="29.7" y2="55.9" width="0.6096" layer="1"/>
+<wire x1="53.8" y1="55.9" x2="42.9" y2="55.9" width="0.6096" layer="1"/>
+<wire x1="42.9" y1="55.9" x2="29.7" y2="55.9" width="0.6096" layer="1"/>
 <wire x1="29.7" y1="55.9" x2="26.9" y2="53.1" width="0.6096" layer="1"/>
 <wire x1="26.9" y1="53.1" x2="26.9" y2="50.1" width="0.6096" layer="1"/>
@@
 <wire x1="30.5" y1="36.6" x2="29.8" y2="37.3" width="0.8128" layer="1"/>
 <wire x1="29.8" y1="37.3" x2="26.5" y2="37.3" width="0.8128" layer="1"/>
+<contactref element="R3" pad="2"/>
+<wire x1="43" y1="54.151" x2="42.9" y2="54.251" width="0.6096" layer="1"/>
+<wire x1="42.9" y1="54.251" x2="42.9" y2="55.9" width="0.6096" layer="1"/>
 <wire x1="48.26" y1="41.91" x2="48.26" y2="41.9735" width="0" layer="19" extent="1-1"/>
 </signal>
@@
 <wire x1="35.7" y1="50.3" x2="36.5" y2="50.3" width="0.6096" layer="1"/>
 <wire x1="57.07" y1="49.53" x2="57.07" y2="50.63" width="0.6096" layer="1"/>
-<wire x1="57.07" y1="50.63" x2="55.7" y2="52" width="0.6096" layer="1"/>
-<wire x1="55.7" y1="52" x2="42.8" y2="52" width="0.6096" layer="1"/>
-<wire x1="42.8" y1="52" x2="42.3" y2="52.5" width="0.6096" layer="1"/>
-<wire x1="42.3" y1="52.5" x2="40.69" y2="52.5" width="0.6096" layer="1"/>
+<wire x1="57.07" y1="50.63" x2="54.9" y2="52.5" width="0.6096" layer="1"/>
+<wire x1="54.9" y1="52.5" x2="40.69" y2="52.5" width="0.6096" layer="1"/>
 <wire x1="40.69" y1="52.5" x2="40.64" y2="52.45" width="0.6096" layer="1"/>
 <wire x1="29.21" y1="52.07" x2="31.74" y2="54.6" width="0.6096" layer="1"/>
@@
 <contactref element="TINY44" pad="6"/>
 <contactref element="ROTARY" pad="1"/>
-<via x="42.5" y="49.7" extent="1-16" drill="0.8" diameter="1.778" shape="octagon"/>
 <via x="42.9" y="45.4" extent="1-16" drill="0.8" diameter="1.4224" shape="octagon"/>
 <wire x1="41.91" y1="41.9735" x2="41.9" y2="41.9835" width="0.6096" layer="1"/>
@@
 <wire x1="41.9" y1="43.1" x2="42.9" y2="44.1" width="0.6096" layer="1"/>
 <wire x1="42.9" y1="44.1" x2="42.9" y2="45.4" width="0.6096" layer="1"/>
-<wire x1="42.5" y1="49.7" x2="42.67" y2="49.53" width="0.8128" layer="1"/>
-<wire x1="42.67" y1="49.53" x2="47.07" y2="49.53" width="0.8128" layer="1"/>
-<wire x1="42.5" y1="49.7" x2="42.9" y2="49.3" width="0.8128" layer="16"/>
-<wire x1="42.9" y1="49.3" x2="42.9" y2="45.4" width="0.8128" layer="16"/>
+<wire x1="42.9" y1="45.4" x2="47.07" y2="49.53" width="0.4064" layer="16"/>
 </signal>
 <signal name="N$14">
